Commit message: Add files via upload

File: urdf/yurtbot.urdf (robot description, URDF)
Before this commit: robot yurtbot, 3 links, 2 joints
Joints:
- removed joint prop_joint1
- removed joint prop_joint2
- added joint joint1: type continuous, parent base_link, child prop1, origin xyz=-0.12713 -0.07122 -0.05281 rpy=0 0 0, axis 0 1 0
- added joint joint2: type continuous, parent base_link, child prop2, origin xyz=0.12713 -0.07122 -0.05281 rpy=0 0 0, axis 0 1 0
